File: Projects/Stork/CoraZ7_conn.sch (KiCad schematic (older format))
At the start: 1 part, among them U33 Digilent-CoraZ7

Commit message: changed position of cora z7 to be at center with cutout to give headroom for ethernet and powerjack
Parts:
- U33: footprint footprint:CoraZ7 -> footprint:CoraZ7_stack
Changed lines of the file:
@@
 F 0 "U33" H 3850 5825 50  0000 C CNN
 F 1 "Digilent-CoraZ7" H 3850 5734 50  0000 C CNN
-F 2 "footprint:CoraZ7" H 3350 2850 50  0001 C CNN
+F 2 "footprint:CoraZ7_stack" H 3350 2850 50  0001 C CNN
 F 3 "" H 3900 1800 50  0001 C CNN
 	1    3850 3750
@@
 	7550 3300 7450 3300
 $Comp
-L power:GND #PWR?
+L power:GND #PWR0150
 U 1 1 5E6743E0
 P 7300 1550
-F 0 "#PWR?" H 7300 1300 50  0001 C CNN
+F 0 "#PWR0150" H 7300 1300 50  0001 C CNN
 F 1 "GND" H 7305 1377 50  0000 C CNN
 F 2 "" H 7300 1550 50  0001 C CNN

Commit message: manually routed power section. library moved internally.
Parts:
- U33: symbol Stork-rescue:Digilent-CoraZ7-Digilent-CoraZ7 -> Stork-rescue:Digilent-CoraZ7-Digilent-CoraZ7-Stork-rescue
Changed lines of the file:
@@
 	3900 2700 4350 2700
 $Comp
-L Stork-rescue:Digilent-CoraZ7-Digilent-CoraZ7 U?
+L Stork-rescue:Digilent-CoraZ7-Digilent-CoraZ7-Stork-rescue U?
 U 1 1 5E33641B
 P 3850 3750

Commit message: renamed project to HPPSI02
Parts:
- U33: symbol Stork-rescue:Digilent-CoraZ7-Digilent-CoraZ7-Stork-rescue -> HPPSI02-rescue:Digilent-CoraZ7-Digilent-CoraZ7-Stork-rescue-Stork-rescue
Changed lines of the file:
@@
 	3900 2700 4350 2700
 $Comp
-L Stork-rescue:Digilent-CoraZ7-Digilent-CoraZ7-Stork-rescue U?
+L HPPSI02-rescue:Digilent-CoraZ7-Digilent-CoraZ7-Stork-rescue-Stork-rescue U?
 U 1 1 5E33641B
 P 3850 3750
