File: Projects/Stork/PMOD_AD2.sch (KiCad schematic (older format))
At the start: 20 parts, among them U1 AD7991YRJZ-1500RL7, U2 AD8608ARZ-SOIC127P600X175-14N

Commit message: changed position of cora z7 to be at center with cutout to give headroom for ethernet and powerjack
Changed lines of the file:
@@
 $Descr A4 11693 8268
 encoding utf-8
-Sheet 20 29
+Sheet 9 29
 Title ""
 Date ""
@@
 AR Path="/5E3D07C7/5E3C35AE/5E34EE27" Ref="U37"  Part="1"
 AR Path="/5E3D07C7/5E3C35B6/5E34EE27" Ref="U39"  Part="1"
-F 0 "U14" H 5075 3825 50  0000 C CNN
+F 0 "U28" H 5075 3825 50  0000 C CNN
 F 1 "AD8608ARZ-SOIC127P600X175-14N" H 5075 3734 50  0000 C CNN
 F 2 "Package_SO:TSSOP-14_4.4x5mm_P0.65mm" H 4750 3750 50  0001 C CNN
@@
 AR Path="/5E3D07C7/5E3C35AE/5E34F9ED" Ref="C171"  Part="1"
 AR Path="/5E3D07C7/5E3C35B6/5E34F9ED" Ref="C181"  Part="1"
-F 0 "C61" H 2765 2046 50  0000 L CNN
+F 0 "C131" H 2765 2046 50  0000 L CNN
 F 1 "10uF" H 2765 1955 50  0000 L CNN
 F 2 "Capacitor_SMD:C_0402_1005Metric" H 2650 2000 50  0001 C CNN
@@
 AR Path="/5E3D07C7/5E3C35AE/5E351096" Ref="C172"  Part="1"
 AR Path="/5E3D07C7/5E3C35B6/5E351096" Ref="C182"  Part="1"
-F 0 "C62" H 3215 2046 50  0000 L CNN
+F 0 "C132" H 3215 2046 50  0000 L CNN
 F 1 "0.1uF" H 3215 1955 50  0000 L CNN
 F 2 "Capacitor_SMD:C_0402_1005Metric" H 3100 2000 50  0001 C CNN
@@
 AR Path="/5E3D07C7/5E3C35AE/5E351172" Ref="#PWR0131"  Part="1"
 AR Path="/5E3D07C7/5E3C35B6/5E351172" Ref="#PWR0137"  Part="1"
-F 0 "#PWR037" H 2650 2250 50  0001 C CNN
+F 0 "#PWR067" H 2650 2250 50  0001 C CNN
 F 1 "GND" H 2655 2327 50  0000 C CNN
 F 2 "" H 2650 2500 50  0001 C CNN
@@
 AR Path="/5E3D07C7/5E3C35AE/5E3514C2" Ref="#PWR0132"  Part="1"
 AR Path="/5E3D07C7/5E3C35B6/5E3514C2" Ref="#PWR0138"  Part="1"
-F 0 "#PWR038" H 4200 2250 50  0001 C CNN
+F 0 "#PWR068" H 4200 2250 50  0001 C CNN
 F 1 "GND" H 4205 2327 50  0000 C CNN
 F 2 "" H 4200 2500 50  0001 C CNN
@@
 AR Path="/5E3D07C7/5E3C35AE/5E354E91" Ref="C173"  Part="1"
 AR Path="/5E3D07C7/5E3C35B6/5E354E91" Ref="C183"  Part="1"
-F 0 "C63" H 7265 1796 50  0000 L CNN
+F 0 "C133" H 7265 1796 50  0000 L CNN
 F 1 "220pF" H 7265 1705 50  0000 L CNN
 F 2 "Capacitor_SMD:C_0402_1005Metric" H 7150 1750 50  0001 C CNN
@@
 AR Path="/5E3D07C7/5E3C35AE/5E355BA6" Ref="C177"  Part="1"
 AR Path="/5E3D07C7/5E3C35B6/5E355BA6" Ref="C187"  Part="1"
-F 0 "C67" V 7502 1200 50  0000 C CNN
+F 0 "C137" V 7502 1200 50  0000 C CNN
 F 1 "470pF" V 7411 1200 50  0000 C CNN
 F 2 "Capacitor_SMD:C_0402_1005Metric" H 7250 1200 50  0001 C CNN
@@
 AR Path="/5E3D07C7/5E3C35AE/5E356132" Ref="R137"  Part="1"
 AR Path="/5E3D07C7/5E3C35B6/5E356132" Ref="R145"  Part="1"
-F 0 "R49" V 7345 1500 50  0000 C CNN
+F 0 "R105" V 7345 1500 50  0000 C CNN
 F 1 "10K" V 7436 1500 50  0000 C CNN
 F 2 "Resistor_SMD:R_0402_1005Metric" V 7590 1490 50  0001 C CNN
@@
 AR Path="/5E3D07C7/5E3C35AE/5E356DA7" Ref="R141"  Part="1"
 AR Path="/5E3D07C7/5E3C35B6/5E356DA7" Ref="R149"  Part="1"
-F 0 "R53" V 7845 1500 50  0000 C CNN
+F 0 "R109" V 7845 1500 50  0000 C CNN
 F 1 "10K" V 7936 1500 50  0000 C CNN
 F 2 "Resistor_SMD:R_0402_1005Metric" V 8090 1490 50  0001 C CNN
@@
 AR Path="/5E3D07C7/5E3C35AE/5E359511" Ref="#PWR0133"  Part="1"
 AR Path="/5E3D07C7/5E3C35B6/5E359511" Ref="#PWR0139"  Part="1"
-F 0 "#PWR039" H 7150 1700 50  0001 C CNN
+F 0 "#PWR069" H 7150 1700 50  0001 C CNN
 F 1 "GND" H 7155 1777 50  0000 C CNN
 F 2 "" H 7150 1950 50  0001 C CNN
@@
 AR Path="/5E3D07C7/5E3C35AE/5E35D840" Ref="C174"  Part="1"
 AR Path="/5E3D07C7/5E3C35B6/5E35D840" Ref="C184"  Part="1"
-F 0 "C64" H 7265 3146 50  0000 L CNN
+F 0 "C134" H 7265 3146 50  0000 L CNN
 F 1 "220pF" H 7265 3055 50  0000 L CNN
 F 2 "Capacitor_SMD:C_0402_1005Metric" H 7150 3100 50  0001 C CNN
@@
 AR Path="/5E3D07C7/5E3C35AE/5E35D846" Ref="C178"  Part="1"
 AR Path="/5E3D07C7/5E3C35B6/5E35D846" Ref="C188"  Part="1"
-F 0 "C68" V 7502 2550 50  0000 C CNN
+F 0 "C138" V 7502 2550 50  0000 C CNN
 F 1 "470pF" V 7411 2550 50  0000 C CNN
 F 2 "Capacitor_SMD:C_0402_1005Metric" H 7250 2550 50  0001 C CNN
@@
 AR Path="/5E3D07C7/5E3C35AE/5E35D84C" Ref="R138"  Part="1"
 AR Path="/5E3D07C7/5E3C35B6/5E35D84C" Ref="R146"  Part="1"
-F 0 "R50" V 7345 2850 50  0000 C CNN
+F 0 "R106" V 7345 2850 50  0000 C CNN
 F 1 "10K" V 7436 2850 50  0000 C CNN
 F 2 "Resistor_SMD:R_0402_1005Metric" V 7590 2840 50  0001 C CNN
@@
 AR Path="/5E3D07C7/5E3C35AE/5E35D852" Ref="R142"  Part="1"
 AR Path="/5E3D07C7/5E3C35B6/5E35D852" Ref="R150"  Part="1"
-F 0 "R54" V 7845 2850 50  0000 C CNN
+F 0 "R110" V 7845 2850 50  0000 C CNN
 F 1 "10K" V 7936 2850 50  0000 C CNN
 F 2 "Resistor_SMD:R_0402_1005Metric" V 8090 2840 50  0001 C CNN
@@
 AR Path="/5E3D07C7/5E3C35AE/5E35D85A" Ref="#PWR0134"  Part="1"
 AR Path="/5E3D07C7/5E3C35B6/5E35D85A" Ref="#PWR0140"  Part="1"
-F 0 "#PWR040" H 7150 3050 50  0001 C CNN
+F 0 "#PWR070" H 7150 3050 50  0001 C CNN
 F 1 "GND" H 7155 3127 50  0000 C CNN
 F 2 "" H 7150 3300 50  0001 C CNN
@@
 AR Path="/5E3D07C7/5E3C35AE/5E360249" Ref="C175"  Part="1"
 AR Path="/5E3D07C7/5E3C35B6/5E360249" Ref="C185"  Part="1"
-F 0 "C65" H 7265 4446 50  0000 L CNN
+F 0 "C135" H 7265 4446 50  0000 L CNN
 F 1 "220pF" H 7265 4355 50  0000 L CNN
 F 2 "Capacitor_SMD:C_0402_1005Metric" H 7150 4400 50  0001 C CNN
@@
 AR Path="/5E3D07C7/5E3C35AE/5E36024F" Ref="C179"  Part="1"
 AR Path="/5E3D07C7/5E3C35B6/5E36024F" Ref="C189"  Part="1"
-F 0 "C69" V 7502 3850 50  0000 C CNN
+F 0 "C139" V 7502 3850 50  0000 C CNN
 F 1 "470pF" V 7411 3850 50  0000 C CNN
 F 2 "Capacitor_SMD:C_0402_1005Metric" H 7250 3850 50  0001 C CNN
@@
 AR Path="/5E3D07C7/5E3C35AE/5E360255" Ref="R139"  Part="1"
 AR Path="/5E3D07C7/5E3C35B6/5E360255" Ref="R147"  Part="1"
-F 0 "R51" V 7345 4150 50  0000 C CNN
+F 0 "R107" V 7345 4150 50  0000 C CNN
 F 1 "10K" V 7436 4150 50  0000 C CNN
 F 2 "Resistor_SMD:R_0402_1005Metric" V 7590 4140 50  0001 C CNN
@@
 AR Path="/5E3D07C7/5E3C35AE/5E36025B" Ref="R143"  Part="1"
 AR Path="/5E3D07C7/5E3C35B6/5E36025B" Ref="R151"  Part="1"
-F 0 "R55" V 7845 4150 50  0000 C CNN
+F 0 "R111" V 7845 4150 50  0000 C CNN
 F 1 "10K" V 7936 4150 50  0000 C CNN
 F 2 "Resistor_SMD:R_0402_1005Metric" V 8090 4140 50  0001 C CNN
@@
 AR Path="/5E3D07C7/5E3C35AE/5E360263" Ref="#PWR0135"  Part="1"
 AR Path="/5E3D07C7/5E3C35B6/5E360263" Ref="#PWR0141"  Part="1"
-F 0 "#PWR041" H 7150 4350 50  0001 C CNN
+F 0 "#PWR071" H 7150 4350 50  0001 C CNN
 F 1 "GND" H 7155 4427 50  0000 C CNN
 F 2 "" H 7150 4600 50  0001 C CNN
@@
 AR Path="/5E3D07C7/5E3C35AE/5E361D85" Ref="C176"  Part="1"
 AR Path="/5E3D07C7/5E3C35B6/5E361D85" Ref="C186"  Part="1"
-F 0 "C66" H 7265 5746 50  0000 L CNN
+F 0 "C136" H 7265 5746 50  0000 L CNN
 F 1 "220pF" H 7265 5655 50  0000 L CNN
 F 2 "Capacitor_SMD:C_0402_1005Metric" H 7150 5700 50  0001 C CNN
@@
 AR Path="/5E3D07C7/5E3C35AE/5E361D8B" Ref="C180"  Part="1"
 AR Path="/5E3D07C7/5E3C35B6/5E361D8B" Ref="C190"  Part="1"
-F 0 "C70" V 7502 5150 50  0000 C CNN
+F 0 "C140" V 7502 5150 50  0000 C CNN
 F 1 "470pF" V 7411 5150 50  0000 C CNN
 F 2 "Capacitor_SMD:C_0402_1005Metric" H 7250 5150 50  0001 C CNN
@@
 AR Path="/5E3D07C7/5E3C35AE/5E361D91" Ref="R140"  Part="1"
 AR Path="/5E3D07C7/5E3C35B6/5E361D91" Ref="R148"  Part="1"
-F 0 "R52" V 7345 5450 50  0000 C CNN
+F 0 "R108" V 7345 5450 50  0000 C CNN
 F 1 "10K" V 7436 5450 50  0000 C CNN
 F 2 "Resistor_SMD:R_0402_1005Metric" V 7590 5440 50  0001 C CNN
@@
 AR Path="/5E3D07C7/5E3C35AE/5E361D97" Ref="R144"  Part="1"
 AR Path="/5E3D07C7/5E3C35B6/5E361D97" Ref="R152"  Part="1"
-F 0 "R56" V 7845 5450 50  0000 C CNN
+F 0 "R112" V 7845 5450 50  0000 C CNN
 F 1 "10K" V 7936 5450 50  0000 C CNN
 F 2 "Resistor_SMD:R_0402_1005Metric" V 8090 5440 50  0001 C CNN
@@
 AR Path="/5E3D07C7/5E3C35AE/5E361D9F" Ref="#PWR0136"  Part="1"
 AR Path="/5E3D07C7/5E3C35B6/5E361D9F" Ref="#PWR0142"  Part="1"
-F 0 "#PWR042" H 7150 5650 50  0001 C CNN
+F 0 "#PWR072" H 7150 5650 50  0001 C CNN
 F 1 "GND" H 7155 5727 50  0000 C CNN
 F 2 "" H 7150 5900 50  0001 C CNN
@@
 AR Path="/5E3D07C7/5E3B1344/5E73DE93" Ref="#PWR0176"  Part="1"
 AR Path="/5E3D07C7/5E3B134C/5E73DE93" Ref="#PWR0177"  Part="1"
-F 0 "#PWR0173" H 2650 1300 50  0001 C CNN
+F 0 "#PWR0160" H 2650 1300 50  0001 C CNN
 F 1 "VDD" H 2667 1623 50  0000 C CNN
 F 2 "" H 2650 1450 50  0001 C CNN
@@
 AR Path="/5E3D07C7/5E3C35AE/5E34EE21" Ref="U36"  Part="1"
 AR Path="/5E3D07C7/5E3C35B6/5E34EE21" Ref="U38"  Part="1"
-F 0 "U13" H 5000 2420 50  0000 C CNN
+F 0 "U27" H 5000 2420 50  0000 C CNN
 F 1 "AD7991YRJZ-1500RL7" H 5000 2329 50  0000 C CNN
 F 2 "Package_TO_SOT_SMD:SOT-23-8" H 5000 1850 50  0001 L BNN
@@
 AR Path="/5E3D07C7/5E3C35AE/5E49DFAB" Ref="#PWR0216"  Part="1"
 AR Path="/5E3D07C7/5E3C35B6/5E49DFAB" Ref="#PWR0217"  Part="1"
-F 0 "#PWR0224" H 6000 3200 50  0001 C CNN
+F 0 "#PWR0230" H 6000 3200 50  0001 C CNN
 F 1 "GND" H 6005 3277 50  0000 C CNN
 F 2 "" H 6000 3450 50  0001 C CNN

Commit message: Pin headers have pins connected to ground
Changed lines of the file:
@@
 $Descr A4 11693 8268
 encoding utf-8
-Sheet 9 29
+Sheet 19 29
 Title ""
 Date ""
@@
 AR Path="/5E3D07C7/5E3C35AE/5E34EE27" Ref="U37"  Part="1"
 AR Path="/5E3D07C7/5E3C35B6/5E34EE27" Ref="U39"  Part="1"
-F 0 "U28" H 5075 3825 50  0000 C CNN
+F 0 "U2" H 5075 3825 50  0000 C CNN
 F 1 "AD8608ARZ-SOIC127P600X175-14N" H 5075 3734 50  0000 C CNN
 F 2 "Package_SO:TSSOP-14_4.4x5mm_P0.65mm" H 4750 3750 50  0001 C CNN
@@
 AR Path="/5E3D07C7/5E3C35AE/5E34F9ED" Ref="C171"  Part="1"
 AR Path="/5E3D07C7/5E3C35B6/5E34F9ED" Ref="C181"  Part="1"
-F 0 "C131" H 2765 2046 50  0000 L CNN
+F 0 "C1" H 2765 2046 50  0000 L CNN
 F 1 "10uF" H 2765 1955 50  0000 L CNN
 F 2 "Capacitor_SMD:C_0402_1005Metric" H 2650 2000 50  0001 C CNN
@@
 AR Path="/5E3D07C7/5E3C35AE/5E351096" Ref="C172"  Part="1"
 AR Path="/5E3D07C7/5E3C35B6/5E351096" Ref="C182"  Part="1"
-F 0 "C132" H 3215 2046 50  0000 L CNN
+F 0 "C2" H 3215 2046 50  0000 L CNN
 F 1 "0.1uF" H 3215 1955 50  0000 L CNN
 F 2 "Capacitor_SMD:C_0402_1005Metric" H 3100 2000 50  0001 C CNN
@@
 AR Path="/5E3D07C7/5E3C35AE/5E351172" Ref="#PWR0131"  Part="1"
 AR Path="/5E3D07C7/5E3C35B6/5E351172" Ref="#PWR0137"  Part="1"
-F 0 "#PWR067" H 2650 2250 50  0001 C CNN
+F 0 "#PWR01" H 2650 2250 50  0001 C CNN
 F 1 "GND" H 2655 2327 50  0000 C CNN
 F 2 "" H 2650 2500 50  0001 C CNN
@@
 AR Path="/5E3D07C7/5E3C35AE/5E3514C2" Ref="#PWR0132"  Part="1"
 AR Path="/5E3D07C7/5E3C35B6/5E3514C2" Ref="#PWR0138"  Part="1"
-F 0 "#PWR068" H 4200 2250 50  0001 C CNN
+F 0 "#PWR02" H 4200 2250 50  0001 C CNN
 F 1 "GND" H 4205 2327 50  0000 C CNN
 F 2 "" H 4200 2500 50  0001 C CNN
@@
 AR Path="/5E3D07C7/5E3C35AE/5E354E91" Ref="C173"  Part="1"
 AR Path="/5E3D07C7/5E3C35B6/5E354E91" Ref="C183"  Part="1"
-F 0 "C133" H 7265 1796 50  0000 L CNN
+F 0 "C3" H 7265 1796 50  0000 L CNN
 F 1 "220pF" H 7265 1705 50  0000 L CNN
 F 2 "Capacitor_SMD:C_0402_1005Metric" H 7150 1750 50  0001 C CNN
@@
 AR Path="/5E3D07C7/5E3C35AE/5E355BA6" Ref="C177"  Part="1"
 AR Path="/5E3D07C7/5E3C35B6/5E355BA6" Ref="C187"  Part="1"
-F 0 "C137" V 7502 1200 50  0000 C CNN
+F 0 "C7" V 7502 1200 50  0000 C CNN
 F 1 "470pF" V 7411 1200 50  0000 C CNN
 F 2 "Capacitor_SMD:C_0402_1005Metric" H 7250 1200 50  0001 C CNN
@@
 AR Path="/5E3D07C7/5E3C35AE/5E356132" Ref="R137"  Part="1"
 AR Path="/5E3D07C7/5E3C35B6/5E356132" Ref="R145"  Part="1"
-F 0 "R105" V 7345 1500 50  0000 C CNN
+F 0 "R1" V 7345 1500 50  0000 C CNN
 F 1 "10K" V 7436 1500 50  0000 C CNN
 F 2 "Resistor_SMD:R_0402_1005Metric" V 7590 1490 50  0001 C CNN
@@
 AR Path="/5E3D07C7/5E3C35AE/5E356DA7" Ref="R141"  Part="1"
 AR Path="/5E3D07C7/5E3C35B6/5E356DA7" Ref="R149"  Part="1"
-F 0 "R109" V 7845 1500 50  0000 C CNN
+F 0 "R5" V 7845 1500 50  0000 C CNN
 F 1 "10K" V 7936 1500 50  0000 C CNN
 F 2 "Resistor_SMD:R_0402_1005Metric" V 8090 1490 50  0001 C CNN
@@
 AR Path="/5E3D07C7/5E3C35AE/5E359511" Ref="#PWR0133"  Part="1"
 AR Path="/5E3D07C7/5E3C35B6/5E359511" Ref="#PWR0139"  Part="1"
-F 0 "#PWR069" H 7150 1700 50  0001 C CNN
+F 0 "#PWR03" H 7150 1700 50  0001 C CNN
 F 1 "GND" H 7155 1777 50  0000 C CNN
 F 2 "" H 7150 1950 50  0001 C CNN
@@
 AR Path="/5E3D07C7/5E3C35AE/5E35D840" Ref="C174"  Part="1"
 AR Path="/5E3D07C7/5E3C35B6/5E35D840" Ref="C184"  Part="1"
-F 0 "C134" H 7265 3146 50  0000 L CNN
+F 0 "C4" H 7265 3146 50  0000 L CNN
 F 1 "220pF" H 7265 3055 50  0000 L CNN
 F 2 "Capacitor_SMD:C_0402_1005Metric" H 7150 3100 50  0001 C CNN
@@
 AR Path="/5E3D07C7/5E3C35AE/5E35D846" Ref="C178"  Part="1"
 AR Path="/5E3D07C7/5E3C35B6/5E35D846" Ref="C188"  Part="1"
-F 0 "C138" V 7502 2550 50  0000 C CNN
+F 0 "C8" V 7502 2550 50  0000 C CNN
 F 1 "470pF" V 7411 2550 50  0000 C CNN
 F 2 "Capacitor_SMD:C_0402_1005Metric" H 7250 2550 50  0001 C CNN
@@
 AR Path="/5E3D07C7/5E3C35AE/5E35D84C" Ref="R138"  Part="1"
 AR Path="/5E3D07C7/5E3C35B6/5E35D84C" Ref="R146"  Part="1"
-F 0 "R106" V 7345 2850 50  0000 C CNN
+F 0 "R2" V 7345 2850 50  0000 C CNN
 F 1 "10K" V 7436 2850 50  0000 C CNN
 F 2 "Resistor_SMD:R_0402_1005Metric" V 7590 2840 50  0001 C CNN
@@
 AR Path="/5E3D07C7/5E3C35AE/5E35D852" Ref="R142"  Part="1"
 AR Path="/5E3D07C7/5E3C35B6/5E35D852" Ref="R150"  Part="1"
-F 0 "R110" V 7845 2850 50  0000 C CNN
+F 0 "R6" V 7845 2850 50  0000 C CNN
 F 1 "10K" V 7936 2850 50  0000 C CNN
 F 2 "Resistor_SMD:R_0402_1005Metric" V 8090 2840 50  0001 C CNN
@@
 AR Path="/5E3D07C7/5E3C35AE/5E35D85A" Ref="#PWR0134"  Part="1"
 AR Path="/5E3D07C7/5E3C35B6/5E35D85A" Ref="#PWR0140"  Part="1"
-F 0 "#PWR070" H 7150 3050 50  0001 C CNN
+F 0 "#PWR04" H 7150 3050 50  0001 C CNN
 F 1 "GND" H 7155 3127 50  0000 C CNN
 F 2 "" H 7150 3300 50  0001 C CNN
@@
 AR Path="/5E3D07C7/5E3C35AE/5E360249" Ref="C175"  Part="1"
 AR Path="/5E3D07C7/5E3C35B6/5E360249" Ref="C185"  Part="1"
-F 0 "C135" H 7265 4446 50  0000 L CNN
+F 0 "C5" H 7265 4446 50  0000 L CNN
 F 1 "220pF" H 7265 4355 50  0000 L CNN
 F 2 "Capacitor_SMD:C_0402_1005Metric" H 7150 4400 50  0001 C CNN
@@
 AR Path="/5E3D07C7/5E3C35AE/5E36024F" Ref="C179"  Part="1"
 AR Path="/5E3D07C7/5E3C35B6/5E36024F" Ref="C189"  Part="1"
-F 0 "C139" V 7502 3850 50  0000 C CNN
+F 0 "C9" V 7502 3850 50  0000 C CNN
 F 1 "470pF" V 7411 3850 50  0000 C CNN
 F 2 "Capacitor_SMD:C_0402_1005Metric" H 7250 3850 50  0001 C CNN
@@
 AR Path="/5E3D07C7/5E3C35AE/5E360255" Ref="R139"  Part="1"
 AR Path="/5E3D07C7/5E3C35B6/5E360255" Ref="R147"  Part="1"
-F 0 "R107" V 7345 4150 50  0000 C CNN
+F 0 "R3" V 7345 4150 50  0000 C CNN
 F 1 "10K" V 7436 4150 50  0000 C CNN
 F 2 "Resistor_SMD:R_0402_1005Metric" V 7590 4140 50  0001 C CNN
@@
 AR Path="/5E3D07C7/5E3C35AE/5E36025B" Ref="R143"  Part="1"
 AR Path="/5E3D07C7/5E3C35B6/5E36025B" Ref="R151"  Part="1"
-F 0 "R111" V 7845 4150 50  0000 C CNN
+F 0 "R7" V 7845 4150 50  0000 C CNN
 F 1 "10K" V 7936 4150 50  0000 C CNN
 F 2 "Resistor_SMD:R_0402_1005Metric" V 8090 4140 50  0001 C CNN
@@
 AR Path="/5E3D07C7/5E3C35AE/5E360263" Ref="#PWR0135"  Part="1"
 AR Path="/5E3D07C7/5E3C35B6/5E360263" Ref="#PWR0141"  Part="1"
-F 0 "#PWR071" H 7150 4350 50  0001 C CNN
+F 0 "#PWR05" H 7150 4350 50  0001 C CNN
 F 1 "GND" H 7155 4427 50  0000 C CNN
 F 2 "" H 7150 4600 50  0001 C CNN
@@
 AR Path="/5E3D07C7/5E3C35AE/5E361D85" Ref="C176"  Part="1"
 AR Path="/5E3D07C7/5E3C35B6/5E361D85" Ref="C186"  Part="1"
-F 0 "C136" H 7265 5746 50  0000 L CNN
+F 0 "C6" H 7265 5746 50  0000 L CNN
 F 1 "220pF" H 7265 5655 50  0000 L CNN
 F 2 "Capacitor_SMD:C_0402_1005Metric" H 7150 5700 50  0001 C CNN
@@
 AR Path="/5E3D07C7/5E3C35AE/5E361D8B" Ref="C180"  Part="1"
 AR Path="/5E3D07C7/5E3C35B6/5E361D8B" Ref="C190"  Part="1"
-F 0 "C140" V 7502 5150 50  0000 C CNN
+F 0 "C10" V 7502 5150 50  0000 C CNN
 F 1 "470pF" V 7411 5150 50  0000 C CNN
 F 2 "Capacitor_SMD:C_0402_1005Metric" H 7250 5150 50  0001 C CNN
@@
 AR Path="/5E3D07C7/5E3C35AE/5E361D91" Ref="R140"  Part="1"
 AR Path="/5E3D07C7/5E3C35B6/5E361D91" Ref="R148"  Part="1"
-F 0 "R108" V 7345 5450 50  0000 C CNN
+F 0 "R4" V 7345 5450 50  0000 C CNN
 F 1 "10K" V 7436 5450 50  0000 C CNN
 F 2 "Resistor_SMD:R_0402_1005Metric" V 7590 5440 50  0001 C CNN
@@
 AR Path="/5E3D07C7/5E3C35AE/5E361D97" Ref="R144"  Part="1"
 AR Path="/5E3D07C7/5E3C35B6/5E361D97" Ref="R152"  Part="1"
-F 0 "R112" V 7845 5450 50  0000 C CNN
+F 0 "R8" V 7845 5450 50  0000 C CNN
 F 1 "10K" V 7936 5450 50  0000 C CNN
 F 2 "Resistor_SMD:R_0402_1005Metric" V 8090 5440 50  0001 C CNN
@@
 AR Path="/5E3D07C7/5E3C35AE/5E361D9F" Ref="#PWR0136"  Part="1"
 AR Path="/5E3D07C7/5E3C35B6/5E361D9F" Ref="#PWR0142"  Part="1"
-F 0 "#PWR072" H 7150 5650 50  0001 C CNN
+F 0 "#PWR06" H 7150 5650 50  0001 C CNN
 F 1 "GND" H 7155 5727 50  0000 C CNN
 F 2 "" H 7150 5900 50  0001 C CNN
@@
 AR Path="/5E3D07C7/5E3B1344/5E73DE93" Ref="#PWR0176"  Part="1"
 AR Path="/5E3D07C7/5E3B134C/5E73DE93" Ref="#PWR0177"  Part="1"
-F 0 "#PWR0160" H 2650 1300 50  0001 C CNN
+F 0 "#PWR0172" H 2650 1300 50  0001 C CNN
 F 1 "VDD" H 2667 1623 50  0000 C CNN
 F 2 "" H 2650 1450 50  0001 C CNN
@@
 AR Path="/5E3D07C7/5E3C35AE/5E34EE21" Ref="U36"  Part="1"
 AR Path="/5E3D07C7/5E3C35B6/5E34EE21" Ref="U38"  Part="1"
-F 0 "U27" H 5000 2420 50  0000 C CNN
+F 0 "U1" H 5000 2420 50  0000 C CNN
 F 1 "AD7991YRJZ-1500RL7" H 5000 2329 50  0000 C CNN
 F 2 "Package_TO_SOT_SMD:SOT-23-8" H 5000 1850 50  0001 L BNN
@@
 AR Path="/5E3D07C7/5E3C35AE/5E49DFAB" Ref="#PWR0216"  Part="1"
 AR Path="/5E3D07C7/5E3C35B6/5E49DFAB" Ref="#PWR0217"  Part="1"
-F 0 "#PWR0230" H 6000 3200 50  0001 C CNN
+F 0 "#PWR0223" H 6000 3200 50  0001 C CNN
 F 1 "GND" H 6005 3277 50  0000 C CNN
 F 2 "" H 6000 3450 50  0001 C CNN
